File: hardware/ASSI/ASSI.kicad_pcb (KiCad board)
At the start: 2 copper layers, 110 x 45 mm, 40 parts

Commit message: Add resistor and capacitor values to ASSI board
- Red: 2 x 300 ohm, green: 1 x 1k, blue: 3 x 43 ohm per LED row
- C3, C4: 100 nF
- Regenerate schematic PDF, images and fabrication output
- Update README with the component values

Co-Authored-By: Claude Opus 5.5 <noreply@anthropic.com>
Parts:
- C3, C4: value C -> 100nF
- R1, R13, R15, R2, R7, R9: value R -> 300
- R10, R16, R3: value R -> 1k
- R11, R12, R14, R17, R18, R4, R5, R6, R8: value R -> 43
Changed lines of the file:
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@@
 			)
 		)
-		(property "Value" "R"
+		(property "Value" "43"
 			(at 0 1.82 0)
 			(layer "F.Fab")
@@
 			)
 		)
-		(property "Value" "C"
+		(property "Value" "100nF"
 			(at 0 1.68 90)
 			(layer "F.Fab")
@@
 			)
 		)
-		(property "Value" "R"
+		(property "Value" "43"
 			(at 0 1.82 0)
 			(layer "F.Fab")
@@
 			)
 		)
-		(property "Value" "R"
+		(property "Value" "300"
 			(at 0 1.82 0)
 			(layer "F.Fab")
@@
 			)
 		)
-		(property "Value" "R"
+		(property "Value" "1k"
 			(at 0 1.82 0)
 			(layer "F.Fab")
@@
 			)
 		)
-		(property "Value" "R"
+		(property "Value" "300"
 			(at 0 1.82 0)
 			(layer "F.Fab")
@@
 			)
 		)
-		(property "Value" "R"
+		(property "Value" "300"
 			(at 0 0 0)
 			(layer "F.Fab")
@@
 			)
 		)
-		(property "Value" "R"
+		(property "Value" "43"
 			(at 0 1.82 0)
 			(layer "F.Fab")
@@
 			)
 		)
-		(property "Value" "R"
+		(property "Value" "43"
 			(at 0 1.82 0)
 			(layer "F.Fab")
@@
 			)
 		)
-		(property "Value" "R"
+		(property "Value" "43"
 			(at 0 1.82 0)
 			(layer "F.Fab")
@@
 			)
 		)
-		(property "Value" "R"
+		(property "Value" "43"
 			(at 0 1.82 0)
 			(layer "F.Fab")
@@
 			)
 		)
-		(property "Value" "R"
+		(property "Value" "1k"
 			(at 0 1.82 0)
 			(layer "F.Fab")
@@
 			)
 		)
-		(property "Value" "R"
+		(property "Value" "300"
 			(at 0 1.82 0)
 			(layer "F.Fab")
@@
 			)
 		)
-		(property "Value" "R"
+		(property "Value" "300"
 			(at 0 1.82 0)
 			(layer "F.Fab")
@@
 			)
 		)
-		(property "Value" "R"
+		(property "Value" "300"
 			(at 0 1.82 0)
 			(layer "F.Fab")
@@
 			)
 		)
-		(property "Value" "R"
+		(property "Value" "43"
 			(at 0 1.82 0)
 			(layer "F.Fab")
@@
 			)
 		)
-		(property "Value" "R"
+		(property "Value" "1k"
 			(at 0 1.82 0)
 			(layer "F.Fab")
@@
 			)
 		)
-		(property "Value" "C"
+		(property "Value" "100nF"
 			(at 0 1.68 90)
 			(layer "F.Fab")
@@
 			)
 		)
-		(property "Value" "R"
+		(property "Value" "43"
 			(at 0 1.82 0)
 			(layer "F.Fab")
@@
 			)
 		)
-		(property "Value" "R"
+		(property "Value" "43"
 			(at 0 1.82 0)
 			(layer "F.Fab")
@@
 			(effects
 				(font
-					(size 1.7 1.7)
+					(size 1.524 1.524)
 					(thickness 0.3)
 				)
@@
 			(effects
 				(font
-					(size 1.65 1.65)
+					(size 1.524 1.524)
 					(thickness 0.3)
 				)

Commit message: Address design review issues on ASSI board
- D1/D2: PMEG4010CEH Schottky (SOD-123F), blue resistors 3 x 47 ohm
- Resistors: Panasonic ERJ-P08 1206 0.66 W, rating in value and MPN,
  derating check against the datasheet in the README
- Footprints from standard KiCad libraries, ISC logo from IFS-KicadLib
- 4 x M3 non-plated mounting holes with 8 mm copper keep-out
- Power net class (0.8 mm) and LED net class (0.5 mm), GND stitching vias
- Manufacturer and MPN fields on every part, bom.csv and positions.csv
- Regenerate schematic PDF, images and fabrication output
- README: rules compliance, mounting configuration, currents and power,
  updated PCB data, BOM with MPNs and open points

Co-Authored-By: Claude Opus 5.5 <noreply@anthropic.com>
Parts:
- added H1: MountingHole, MountingHole:MountingHole_3.2mm_M3, F.Cu at (96.0, 72.0)
- added H2: MountingHole, MountingHole:MountingHole_3.2mm_M3, F.Cu at (96.0, 107.0)
- added H3: MountingHole, MountingHole:MountingHole_3.2mm_M3, F.Cu at (196.0, 72.0)
- added H4: MountingHole, MountingHole:MountingHole_3.2mm_M3, F.Cu at (196.0, 107.0)
- D1, D2: value 1N914BWS -> PMEG4010CEH; footprint PCM_Diode_SMD_AKL:D_SOD-323F -> Diode_SMD:D_SOD-123F
- G3: footprint Logo_ISC:LogoISC -> ISC_mecanica:LogoISC
- R1, R13, R15, R2, R7, R9: value 300 -> 300R 1% 0.66W; footprint PCM_Resistor_SMD_AKL:R_1206_3216Metric_Pad1.30x1.75mm_HandSolder -> Resistor_SMD:R_1206_3216Metric_Pad1.30x1.75mm_HandSolder
- R10, R16, R3: value 1k -> 1k 1% 0.66W; footprint PCM_Resistor_SMD_AKL:R_1206_3216Metric_Pad1.30x1.75mm_HandSolder -> Resistor_SMD:R_1206_3216Metric_Pad1.30x1.75mm_HandSolder
- R11, R12, R14, R17, R18, R4, R5, R6, R8: value 43 -> 47R 1% 0.66W; footprint PCM_Resistor_SMD_AKL:R_1206_3216Metric_Pad1.30x1.75mm_HandSolder -> Resistor_SMD:R_1206_3216Metric_Pad1.30x1.75mm_HandSolder
- moved OUT1 0.50 mm to (193.5, 86.5)
Routing:
- net GND: track 6.81 -> 6.86 mm, vias 0 -> 15
